File: Documentation/Electrical/PCB/Sources/Battery_Management/Battery_Management/Battery_Management.kicad_sch (KiCad schematic)
At the start: 12 parts, among them J1 AC_P, J2 AC_N, J3 AC_GND, J4 Wall_Socket, J5 Chassis_Int_Socket, J6 Cable_Female, J7 Battery_Conn, P1 Chassis_Ext_Conn, P2 Cable_Male, P3 Power_Conn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

Commit message: Added to batt manage signoff
Parts:
- added J8: Chassis_Int_Socket, symbol Connector:Conn_WallSocket_Earth
- added J9: Cable_Female, symbol Connector:Conn_WallSocket_Earth
- added P4: Chassis_Int_Conn, symbol Connector:Conn_WallPlug_Earth
- added P5: Cable_Male, symbol Connector:Conn_WallPlug_Earth
Connections:
- net at P1.1 (AC_P): now also P4.1 (AC_P); no longer J5.1 (AC_P)
- net at P1.2 (AC_N): now also P4.2 (AC_N); no longer J5.2 (AC_N)
- net at P1.3 (EARTH): now also P4.3 (EARTH); no longer J5.3 (EARTH)
- new net: J5.1 (AC_P), J8.1 (AC_P)
- new net: J5.2 (AC_N), J8.2 (AC_N)
- new net: J5.3 (EARTH), J8.3 (EARTH)
- new net: J9.1 (AC_P), P5.1 (AC_P)
- new net: J9.2 (AC_N), P5.2 (AC_N)
- new net: J9.3 (EARTH), P5.3 (EARTH)
Other:
- note added: "Adapter to connect chassis-mount connector to charger cable IEC 320 C13 - IEC 320 C13"
- note added: "Cable Connecting Battery Charger to Adapter IEC 320 C13 - IEC 320 C14"
- note added: "Cable Connecting wall socket to robot chassis connector NEMA 5-15P - IEC 320 C13"
- note added: "Chassis-mounted power connector IEC 320 C14 - IEC 320 C14"
- note added: "IEC 320 C14 Connector on exterior of battery charger"
- note removed: "Chassis-mounted 3-prong connector"
- moved on the sheet: BT1, J5, J7, P1, P3, U1
